File: schematics/schematics.kicad_pcb (KiCad board)
At the start: 2 copper layers, 40 x 40 mm, 15 parts, among them U1 LTC4124, U2 nRF52832-QFxx, Y1 32mHz

Commit message: assigned 3d models, pcb dev
Parts:
- added C10: 1u, Capacitor_SMD:C_0402_1005Metric, B.Cu at (76.7, 78.1)
- added C11: 0.1u, Capacitor_SMD:C_0402_1005Metric, B.Cu at (89.0, 62.1)
- added C12: 0.1u, Capacitor_SMD:C_0402_1005Metric, B.Cu at (82.2, 74.6)
- added D1: MCL4148, Diode_SMD:D_MicroMELF, B.Cu at (81.5, 57.7)
- added D2: LED_Indicator, LED_SMD:LED_0402_1005Metric, F.Cu at (92.8, 50.5)
- added R1: 1M, Resistor_SMD:R_0402_1005Metric, B.Cu at (80.5, 72.2)
- added R2: 100k, Resistor_SMD:R_0402_1005Metric, B.Cu at (84.3, 58.4)
- added R3: 220, Resistor_SMD:R_0402_1005Metric, B.Cu at (95.7, 56.3)
- added SW1: Button, Button_Switch_SMD:SW_DIP_SPSTx02_Slide_6.7x6.64mm_W6.73mm_P2.54mm_LowProfile_JPin, F.Cu at (92.7, 69.8)
- added U3: TPS22929D, Package_TO_SOT_SMD:SOT-23-6, B.Cu at (89.9, 58.4)
- BT1, C1, C2, C3, C4, C5, C6, C7, C8, C9, L2, U1, U2: moved to B.Cu
- L1: footprint Inductor_SMD:L_0402_1005Metric -> Inductor_SMD:L_TDK_SLF6025; moved to B.Cu
- Y1: footprint Crystal:Crystal_SMD_2016-4Pin_2.0x1.6mm -> Crystal:Crystal_SMD_2012-2Pin_2.0x1.2mm; moved to B.Cu
- moved C2 26.2 mm to (91.7, 85.9)
- moved Y1 23.2 mm to (99.7, 82.6)
- moved C1 20.9 mm to (85.5, 84.0), turned to 270 degrees
- moved C8 15.2 mm to (96.5, 77.5)
- moved C9 14.6 mm to (76.2, 63.9), turned to 90 degrees
- moved U2 11.9 mm to (101.0, 60.1)
- moved L2 10.6 mm to (106.6, 64.8)
- moved C3 10.5 mm to (102.1, 75.9)
- moved C7 10.4 mm to (92.7, 76.2), turned to 90 degrees
- moved C5 10.2 mm to (105.8, 74.1)
- moved BT1 8.29 mm to (74.9, 71.6)
- moved L1 8.28 mm to (92.7, 69.8), turned to 90 degrees
- moved C4 7.85 mm to (105.9, 69.8)
- moved U1 5.97 mm to (84.3, 69.5), turned to 90 degrees
- moved C6 4.39 mm to (101.6, 71.1)
Connections:
- C9 pad 2: /VDD_NRF -> /V_SUP
- U1 pad 1: /VDD_NRF -> /V_LIPOL
- U1 pad 2: /VDD_NRF -> /V_LIPOL
- U1 pad 3: /VDD_NRF -> /V_LIPOL
- U1 pad 4: /VDD_NRF -> /V_LIPOL
- U2 pad 13: /VDD_NRF -> /V_SUP
- U2 pad 36: /VDD_NRF -> /V_SUP
- U2 pad 4: Net-(U2-Pad4) -> /MCU_BTN
- U2 pad 48: /VDD_NRF -> /V_SUP
- U2 pad 8: Net-(U2-Pad8) -> /MCU_PWR
Routing:
- net Net-(D2-Pad2): track 0.00 -> 6.24 mm, vias 0 -> 1
- net Net-(R3-Pad2): track 0.00 -> 4.21 mm
- net GND: track 0.00 -> 1.18 mm

Commit message: pcb development
Parts:
- SW1: footprint Button_Switch_SMD:SW_DIP_SPSTx02_Slide_6.7x6.64mm_W6.73mm_P2.54mm_LowProfile_JPin -> Button_Switch_SMD:SW_SPST_PTS645
- moved BT1 31.2 mm to (105.1, 79.3), turned to 180 degrees
- moved C2 25.9 mm to (104.5, 63.4), turned to 180 degrees
- moved U1 24.0 mm to (108.3, 69.7), turned to 270 degrees
- moved C9 20.4 mm to (94.4, 54.5), turned to 0 degrees
- moved C1 20.1 mm to (100.0, 70.0)
- moved Y1 18.5 mm to (102.4, 64.3), turned to 270 degrees
- moved D1 13.4 mm to (85.5, 70.5)
- moved R1 13.2 mm to (87.7, 61.1), turned to 90 degrees
- moved C8 13.0 mm to (97.1, 64.5)
- moved C7 13.0 mm to (91.9, 63.3), turned to 180 degrees
- moved U3 12.4 mm to (82.0, 68.0)
- moved C5 12.4 mm to (104.9, 61.7), turned to 270 degrees
- moved C10 10.7 mm to (78.3, 67.5), turned to 270 degrees
- moved C3 10.5 mm to (104.5, 65.7)
- moved C12 10.3 mm to (85.5, 64.9), turned to 90 degrees
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Connections:
- C12 pad 1: /VSUP -> /V_SUP
- D1 pad 1: /VSUP -> /V_SUP
- U3 pad 1: /VSUP -> /V_SUP
Routing:
- net GND: track 1.18 -> 58.3 mm, vias 0 -> 1
- net /V_LIPOL: track 0.00 -> 47.8 mm, vias 0 -> 2
- net /V_SUP: track 0.00 -> 39.8 mm, vias 0 -> 4
- net Net-(D1-Pad2): track 0.00 -> 26.2 mm, vias 0 -> 2
- net /MCU_PWR: track 0.00 -> 18.6 mm, vias 0 -> 2
- net Net-(C1-Pad1): track 0.00 -> 15.3 mm
- net Net-(BT1-Pad1): track 0.00 -> 10.4 mm
- net Net-(C4-Pad1): track 0.00 -> 8.49 mm
- net Net-(C3-Pad2): track 0.00 -> 6.23 mm
- net Net-(C5-Pad1): track 0.00 -> 5.77 mm
- net Net-(C2-Pad2): track 0.00 -> 5.27 mm
- net /MCU_BTN: track 0.00 -> 4.31 mm
- net Net-(C7-Pad1): track 0.00 -> 2.34 mm
- net Net-(C6-Pad1): track 0.00 -> 2.33 mm
- net Net-(C8-Pad2): track 0.00 -> 2.07 mm
- added copper zone on B.Cu, net GND
