File: schematics/schematics.sch (KiCad schematic (older format))
At the start: 18 parts

Commit message: schematics development
Parts:
- removed BT?: 4.2V, symbol Device:Battery_Cell
- removed C? (x2): 12pF, symbol Device:C_Small
- removed Y?: 32.768kHz, symbol Device:Crystal_Small
- added BT1: +4.2V, Connector_PinHeader_1.00mm:PinHeader_1x02_P1.00mm_Horizontal, symbol Connector:Conn_01x02_Male
- C1, C2, C3, C4, C5, C6, C7, C8, C9: renamed from C?; footprint (none) -> Capacitor_SMD:C_0402_1005Metric
- L1, L2: renamed from L?; footprint (none) -> Inductor_SMD:L_0402_1005Metric
- Y1: renamed from Y?; footprint (none) -> Crystal:Crystal_SMD_2012-2Pin_2.0x1.2mm
- gave numbers to parts that had none: 2
Connections:
- wire segments 89 -> 79
Changed lines of the file:
@@
 У платы nrf нет некоторых пинов: vdd и vss указаны только один раз\nПеред подключением питание к nrf должен быть Back boost converter
 $Comp
-L Device:Battery_Cell BT?
-U 1 1 5EE68AB4
-P 2400 2550
-F 0 "BT?" H 2450 2650 50  0000 L CNN
-F 1 "4.2V" H 2450 2550 50  0000 L CNN
-F 2 "" V 2400 2610 50  0001 C CNN
-F 3 "~" V 2400 2610 50  0001 C CNN
-	1    2400 2550
-	1    0    0    -1
-$EndComp
-$Comp
-L smart~ring:LTC4124 U?
-U 1 1 5EE74933
-P 2400 1800
-F 0 "U?" H 2400 2417 50  0000 C CNN
-F 1 "LTC4124" H 2400 2326 50  0000 C CNN
-F 2 "Package_DFN_QFN:QFN-12-1EP_3x3mm_P0.5mm_EP1.65x1.65mm" H 2400 700 50  0001 C CNN
-F 3 "" H 2400 600 50  0001 C CNN
-	1    2400 1800
-	1    0    0    -1
-$EndComp
-$Comp
-L power:GND #PWR?
+L power:GND #PWR0101
 U 1 1 5EE792B4
 P 2150 2800
-F 0 "#PWR?" H 2150 2550 50  0001 C CNN
+F 0 "#PWR0101" H 2150 2550 50  0001 C CNN
 F 1 "GND" H 2155 2627 50  0000 C CNN
 F 2 "" H 2150 2800 50  0001 C CNN
@@
 $EndComp
 Wire Wire Line
-	2400 2350 2400 2300
-Wire Wire Line
 	2650 2300 2650 2750
-Wire Wire Line
-	2650 2750 2400 2750
-Wire Wire Line
-	2400 2650 2400 2750
-Connection ~ 2400 2750
-Wire Wire Line
-	2400 2750 2150 2750
 Wire Wire Line
 	2150 2800 2150 2750
@@
 	1800 1650 1800 1750
 $Comp
-L Device:L_Small L?
+L Device:L_Small L1
 U 1 1 5EE93CB8
 P 1200 1950
-F 0 "L?" H 1156 1904 50  0000 R CNN
+F 0 "L1" H 1156 1904 50  0000 R CNN
 F 1 "sm" H 1156 1995 50  0000 R CNN
-F 2 "" H 1200 1950 50  0001 C CNN
+F 2 "Inductor_SMD:L_0402_1005Metric" H 1200 1950 50  0001 C CNN
 F 3 "~" H 1200 1950 50  0001 C CNN
 	1    1200 1950
@@
 $EndComp
 $Comp
-L Device:C_Small C?
+L Device:C_Small C1
 U 1 1 5EE940F1
 P 1450 1950
-F 0 "C?" H 1542 1996 50  0000 L CNN
+F 0 "C1" H 1542 1996 50  0000 L CNN
 F 1 "sm" H 1542 1905 50  0000 L CNN
-F 2 "" H 1450 1950 50  0001 C CNN
+F 2 "Capacitor_SMD:C_0402_1005Metric" H 1450 1950 50  0001 C CNN
 F 3 "~" H 1450 1950 50  0001 C CNN
 	1    1450 1950
@@
 	3000 1650 3000 1750
 $Comp
-L MCU_Nordic:nRF52832-QFxx U?
+L MCU_Nordic:nRF52832-QFxx U2
 U 1 1 5EDD8BEA
 P 8050 3600
-F 0 "U?" H 8750 1900 50  0000 C CNN
+F 0 "U2" H 8750 1900 50  0000 C CNN
 F 1 "nRF52832-QFxx" H 8550 1800 50  0000 C CNN
 F 2 "Package_DFN_QFN:QFN-48-1EP_6x6mm_P0.4mm_EP4.6x4.6mm" H 8050 1500 50  0001 C CNN
@@
 	7550 1900 7550 1800
 $Comp
-L power:GND #PWR?
+L power:GND #PWR0102
 U 1 1 5EDDC9EC
 P 7050 1850
-F 0 "#PWR?" H 7050 1600 50  0001 C CNN
+F 0 "#PWR0102" H 7050 1600 50  0001 C CNN
 F 1 "GND" H 7055 1677 50  0000 C CNN
 F 2 "" H 7050 1850 50  0001 C CNN
@@
 $EndComp
 $Comp
-L Device:C_Small C?
+L Device:C_Small C7
 U 1 1 5EDDD2B2
 P 7300 1800
-F 0 "C?" V 7200 1800 50  0000 C CNN
+F 0 "C7" V 7200 1800 50  0000 C CNN
 F 1 "100nF" V 7400 1800 50  0000 C CNN
-F 2 "" H 7300 1800 50  0001 C CNN
+F 2 "Capacitor_SMD:C_0402_1005Metric" H 7300 1800 50  0001 C CNN
 F 3 "~" H 7300 1800 50  0001 C CNN
 	1    7300 1800
@@
 	7200 1800 7050 1800
 $Comp
-L Device:C_Small C?
-U 1 1 5EDE11A0
-P 10100 1750
-F 0 "C?" V 9871 1750 50  0000 C CNN
-F 1 "12pF" V 9962 1750 50  0000 C CNN
-F 2 "" H 10100 1750 50  0001 C CNN
-F 3 "~" H 10100 1750 50  0001 C CNN
-	1    10100 1750
-	0    1    1    0
-$EndComp
-$Comp
-L Device:C_Small C?
-U 1 1 5EDE14FF
-P 10100 2200
-F 0 "C?" V 9871 2200 50  0000 C CNN
-F 1 "12pF" V 9962 2200 50  0000 C CNN
-F 2 "" H 10100 2200 50  0001 C CNN
-F 3 "~" H 10100 2200 50  0001 C CNN
-	1    10100 2200
-	0    1    1    0
-$EndComp
-$Comp
-L power:GND #PWR?
-U 1 1 5EDE183D
-P 10350 2250
-F 0 "#PWR?" H 10350 2000 50  0001 C CNN
-F 1 "GND" H 10355 2077 50  0000 C CNN
-F 2 "" H 10350 2250 50  0001 C CNN
-F 3 "" H 10350 2250 50  0001 C CNN
-	1    10350 2250
-	1    0    0    -1
-$EndComp
-Wire Wire Line
-	10350 2250 10350 2200
-Wire Wire Line
-	10350 2200 10200 2200
-Wire Wire Line
-	10200 1750 10350 1750
-Wire Wire Line
-	10350 1750 10350 2200
-Connection ~ 10350 2200
-Wire Wire Line
-	10000 2200 9900 2200
-Wire Wire Line
-	10000 1750 9900 1750
-$Comp
-L Device:Crystal_Small Y?
-U 1 1 5EDE5739
-P 9900 2000
-F 0 "Y?" V 9854 2088 50  0000 L CNN
-F 1 "32.768kHz" V 9945 2088 50  0000 L CNN
-F 2 "" H 9900 2000 50  0001 C CNN
-F 3 "~" H 9900 2000 50  0001 C CNN
-	1    9900 2000
-	0    -1   1    0
-$EndComp
-Wire Wire Line
-	9900 1900 9900 1750
-Wire Wire Line
-	9900 2100 9900 2200
-Wire Wire Line
-	8950 2200 9900 2200
-Connection ~ 9900 2200
-Wire Wire Line
-	8950 2100 9200 2100
-Wire Wire Line
-	9200 2100 9200 1750
-Wire Wire Line
-	9200 1750 9900 1750
-Connection ~ 9900 1750
-$Comp
-L Device:C_Small C?
+L Device:C_Small C9
 U 1 1 5EDF5D8F
 P 8450 1650
-F 0 "C?" V 8250 1650 50  0000 C CNN
+F 0 "C9" V 8250 1650 50  0000 C CNN
 F 1 "100nF" V 8350 1700 50  0000 C CNN
-F 2 "" H 8450 1650 50  0001 C CNN
+F 2 "Capacitor_SMD:C_0402_1005Metric" H 8450 1650 50  0001 C CNN
 F 3 "~" H 8450 1650 50  0001 C CNN
 	1    8450 1650
@@
 $EndComp
 $Comp
-L power:GND #PWR?
+L power:GND #PWR0104
 U 1 1 5EDFE067
 P 8550 1750
-F 0 "#PWR?" H 8550 1500 50  0001 C CNN
+F 0 "#PWR0104" H 8550 1500 50  0001 C CNN
 F 1 "GND" H 8555 1577 50  0000 C CNN
 F 2 "" H 8550 1750 50  0001 C CNN
@@
 	8050 5500 8050 5300
 $Comp
-L Device:L_Small L?
+L Device:L_Small L2
 U 1 1 5EE09D8A
 P 6350 2600
-F 0 "L?" V 6535 2600 50  0000 C CNN
+F 0 "L2" V 6535 2600 50  0000 C CNN
 F 1 "3.9nH" V 6444 2600 50  0000 C CNN
-F 2 "" H 6350 2600 50  0001 C CNN
+F 2 "Inductor_SMD:L_0402_1005Metric" H 6350 2600 50  0001 C CNN
 F 3 "~" H 6350 2600 50  0001 C CNN
 	1    6350 2600
@@
 	6250 2600 5950 2600
 $Comp
-L Device:C_Small C?
+L Device:C_Small C4
 U 1 1 5EE0E458
 P 6600 2750
-F 0 "C?" H 6692 2796 50  0000 L CNN
+F 0 "C4" H 6692 2796 50  0000 L CNN
 F 1 "0.8pF" H 6692 2705 50  0000 L CNN
-F 2 "" H 6600 2750 50  0001 C CNN
+F 2 "Capacitor_SMD:C_0402_1005Metric" H 6600 2750 50  0001 C CNN
 F 3 "~" H 6600 2750 50  0001 C CNN
 	1    6600 2750
@@
 	6600 2600 6450 2600
 $Comp
-L power:GND #PWR?
+L power:GND #PWR0105
 U 1 1 5EE1053F
 P 6600 2950
-F 0 "#PWR?" H 6600 2700 50  0001 C CNN
+F 0 "#PWR0105" H 6600 2700 50  0001 C CNN
 F 1 "GND" H 6605 2777 50  0000 C CNN
 F 2 "" H 6600 2950 50  0001 C CNN
@@
 	7000 2900 7000 2600
 $Comp
-L Device:C_Small C?
+L Device:C_Small C6
 U 1 1 5EE1C7C7
 P 7300 1400
-F 0 "C?" V 7200 1400 50  0000 C CNN
+F 0 "C6" V 7200 1400 50  0000 C CNN
 F 1 "N.C." V 7400 1400 50  0000 C CNN
-F 2 "" H 7300 1400 50  0001 C CNN
+F 2 "Capacitor_SMD:C_0402_1005Metric" H 7300 1400 50  0001 C CNN
 F 3 "~" H 7300 1400 50  0001 C CNN
 	1    7300 1400
@@
 $EndComp
 $Comp
-L Device:C_Small C?
+L Device:C_Small C5
 U 1 1 5EE1E35F
 P 7300 1050
-F 0 "C?" V 7200 1050 50  0000 C CNN
+F 0 "C5" V 7200 1050 50  0000 C CNN
 F 1 "100pF" V 7400 1050 50  0000 C CNN
-F 2 "" H 7300 1050 50  0001 C CNN
+F 2 "Capacitor_SMD:C_0402_1005Metric" H 7300 1050 50  0001 C CNN
 F 3 "~" H 7300 1050 50  0001 C CNN
 	1    7300 1050
@@
 	6200 3700 6200 3800
 $Comp
-L Device:Crystal_Small Y?
+L Device:Crystal_Small Y1
 U 1 1 5EE36C8A
 P 6200 3600
-F 0 "Y?" V 6154 3688 50  0000 L CNN
+F 0 "Y1" V 6154 3688 50  0000 L CNN
 F 1 "32mHz" V 6245 3688 50  0000 L CNN
-F 2 "" H 6200 3600 50  0001 C CNN
+F 2 "Crystal:Crystal_SMD_2012-2Pin_2.0x1.2mm" H 6200 3600 50  0001 C CNN
 F 3 "~" H 6200 3600 50  0001 C CNN
 	1    6200 3600
@@
 	6100 3800 6200 3800
 $Comp
-L Device:C_Small C?
+L Device:C_Small C3
 U 1 1 5EE36C77
 P 6000 3800
-F 0 "C?" V 5771 3800 50  0000 C CNN
+F 0 "C3" V 5771 3800 50  0000 C CNN
 F 1 "12pF" V 5862 3800 50  0000 C CNN
-F 2 "" H 6000 3800 50  0001 C CNN
+F 2 "Capacitor_SMD:C_0402_1005Metric" H 6000 3800 50  0001 C CNN
 F 3 "~" H 6000 3800 50  0001 C CNN
 	1    6000 3800
@@
 $EndComp
 $Comp
-L Device:C_Small C?
+L Device:C_Small C2
 U 1 1 5EE36C71
 P 6000 3400
-F 0 "C?" V 5771 3400 50  0000 C CNN
+F 0 "C2" V 5771 3400 50  0000 C CNN
 F 1 "12pF" V 5862 3400 50  0000 C CNN
-F 2 "" H 6000 3400 50  0001 C CNN
+F 2 "Capacitor_SMD:C_0402_1005Metric" H 6000 3400 50  0001 C CNN
 F 3 "~" H 6000 3400 50  0001 C CNN
 	1    6000 3400
@@
 	8050 1900 8050 1650
 $Comp
-L Device:C_Small C?
+L Device:C_Small C8
 U 1 1 5EE5B8DE
 P 8450 1050
-F 0 "C?" V 8250 1050 50  0000 C CNN
+F 0 "C8" V 8250 1050 50  0000 C CNN
 F 1 "1.0μF" V 8350 1100 50  0000 C CNN
-F 2 "" H 8450 1050 50  0001 C CNN
+F 2 "Capacitor_SMD:C_0402_1005Metric" H 8450 1050 50  0001 C CNN
 F 3 "~" H 8450 1050 50  0001 C CNN
 	1    8450 1050
@@
 $EndComp
 $Comp
-L power:GND #PWR?
+L power:GND #PWR0106
 U 1 1 5EE5B8E4
 P 8550 1150
-F 0 "#PWR?" H 8550 900 50  0001 C CNN
+F 0 "#PWR0106" H 8550 900 50  0001 C CNN
 F 1 "GND" H 8555 977 50  0000 C CNN
 F 2 "" H 8550 1150 50  0001 C CNN
@@
 	5900 3400 5750 3400
 $Comp
-L power:GND #PWR?
+L power:GND #PWR0107
 U 1 1 5EE36C7D
 P 5750 3850
-F 0 "#PWR?" H 5750 3600 50  0001 C CNN
+F 0 "#PWR0107" H 5750 3600 50  0001 C CNN
 F 1 "GND" H 5755 3677 50  0000 C CNN
 F 2 "" H 5750 3850 50  0001 C CNN
@@
 Wire Wire Line
 	5750 3800 5900 3800
+$Comp
+L Connector:Conn_01x02_Male BT1
+U 1 1 5EDCCF2E
+P 2250 2450
+F 0 "BT1" H 2300 2500 50  0000 C CNN
+F 1 "+4.2V" H 2300 2300 50  0000 C CNN
+F 2 "Connector_PinHeader_1.00mm:PinHeader_1x02_P1.00mm_Horizontal" H 2250 2450 50  0001 C CNN
+F 3 "~" H 2250 2450 50  0001 C CNN
+	1    2250 2450
+	1    0    0    -1
+$EndComp
+$Comp
+L smart~ring:LTC4124 U1
+U 1 1 5EE74933
+P 2400 1800
+F 0 "U1" H 2400 2417 50  0000 C CNN
+F 1 "LTC4124" H 2400 2326 50  0000 C CNN
+F 2 "Package_DFN_QFN:QFN-12-1EP_3x3mm_P0.5mm_EP1.65x1.65mm" H 2400 700 50  0001 C CNN
+F 3 "" H 2400 600 50  0001 C CNN
+	1    2400 1800
+	1    0    0    -1
+$EndComp
+Wire Wire Line
+	2150 2750 2450 2750
+Wire Wire Line
+	2450 2450 2450 2350
+Wire Wire Line
+	2450 2350 2400 2350
+Wire Wire Line
+	2400 2350 2400 2300
+Wire Wire Line
+	2450 2550 2450 2750
+Connection ~ 2450 2750
+Wire Wire Line
+	2450 2750 2650 2750
 $EndSCHEMATC

Commit message: assigned 3d models, pcb dev
Parts:
- added C10: 1u, Capacitor_SMD:C_0402_1005Metric, symbol Device:C_Small
- added C11, C12: 0.1u, Capacitor_SMD:C_0402_1005Metric, symbol Device:C_Small
- added D1: MCL4148, Diode_SMD:D_MicroMELF, symbol Diode:MCL4148
- added D2: LED_Indicator, LED_SMD:LED_0402_1005Metric, symbol Device:LED_Small_ALT
- added R1: 1M, Resistor_SMD:R_0402_1005Metric, symbol Device:R_Small
- added R2: 100k, Resistor_SMD:R_0402_1005Metric, symbol Device:R_Small
- added R3: 220, Resistor_SMD:R_0402_1005Metric, symbol Device:R_Small
- added SW1: Button, Button_Switch_SMD:SW_DIP_SPSTx02_Slide_6.7x6.64mm_W6.73mm_P2.54mm_LowProfile_JPin, symbol Switch:SW_DPST_x2
- added U3: TPS22929D, Package_TO_SOT_SMD:SOT-23-6, symbol smart~ring:TPS22929D
- L1: footprint Inductor_SMD:L_0402_1005Metric -> Inductor_SMD:L_TDK_SLF6025
Connections:
- net labels added: MCU_BTN, MCU_PWR, VSUP, V_LIPOL, V_SUP
- net labels removed: VDD_NRF
- wire segments 79 -> 118
Other:
- note added: "У платы nrf нет некоторых пинов: vdd и vss указаны только один раз\nПеред подключением питание к nrf должен быть Back boost converter\nПроверить, что mcu_pwr, mcu_btn и led подключены к правильным портам"
- note removed: "У платы nrf нет некоторых пинов: vdd и vss указаны только один раз\nПеред подключением питание к nrf должен быть Back boost converter"
- moved on the sheet: C2, C3, C4, C5, C6, C7, C8, C9, L2, U2, Y1

Commit message: pcb development
Connections:
- net labels removed: VSUP
Changed lines of the file:
@@
 	3300 5150 3950 5150
 Text Label 3950 4950 2    50   ~ 0
-VSUP
+V_SUP
 Wire Wire Line
 	3950 4950 3450 4950
